Commit message: changed knee to shin transformation from fixed to continuout

File: urdf/cassie_with_sensors.urdf (robot description, URDF)
Before this commit: robot cassie, 19 links, 18 joints
Joints:
- removed joint fixed_knee_to_shin_left
- removed joint fixed_knee_to_shin_right
- added joint knee_to_shin_left: type continuous, parent left_knee, child left_shin, origin xyz=0.0607 0.0474 0 rpy=0 0 0, axis 0 0 1, limit lower=-100 upper=100 effort=0 velocity=100
- added joint knee_to_shin_right: type continuous, parent right_knee, child right_shin, origin xyz=0.0607 0.0474 0 rpy=0 0 0, axis 0 0 1, limit lower=-100 upper=100 effort=0 velocity=100

File: urdf/cassie_with_sensors.xacro (robot description, xacro)
@@ -40,5 +40,5 @@
   <xacro:hip_flexion side="left"/>
   <xacro:knee_joint side="left" reflect="1"/>
-  <xacro:fixed_knee_to_shin side="left"/>
+  <xacro:knee_to_shin side="left"/>
   <xacro:ankle_joint side="left"/>
   <xacro:toe_joint side="left"/>
@@ -48,5 +48,5 @@
   <xacro:hip_flexion side="right"/>
   <xacro:knee_joint side="right" reflect="-1"/>
-  <xacro:fixed_knee_to_shin side="right"/>
+  <xacro:knee_to_shin side="right"/>
   <xacro:ankle_joint side="right"/>
   <xacro:toe_joint side="right"/>
@@ -285,5 +285,5 @@
       <parent link="${side}_pelvis_rotation" />
       <child link="${side}_hip" />
-	  <limit lower="-0.3927" upper="0.3927" effort="4.5" velocity="12.1475" />
+      <limit lower="-0.3927" upper="0.3927" effort="4.5" velocity="12.1475" />
     </joint>
   </xacro:macro>
@@ -294,5 +294,5 @@
       <parent link="${side}_hip" />
       <child link="${side}_thigh" />
-	  <limit lower="-0.8727" upper="1.3963" effort="12.2" velocity="8.5085" />
+      <limit lower="-0.8727" upper="1.3963" effort="12.2" velocity="8.5085" />
     </joint>
   </xacro:macro>
@@ -303,14 +303,14 @@
       <parent link="${side}_thigh" />
       <child link="${side}_knee" />
-	  <limit lower="-2.8623" upper="-0.6458" effort="12.2" velocity="8.5085" />
-    </joint>
-  </xacro:macro>
-  <xacro:macro name="fixed_knee_to_shin" params="side">
-    <joint name="fixed_knee_to_shin_${side}" type="fixed">
+      <limit lower="-2.8623" upper="-0.6458" effort="12.2" velocity="8.5085" />
+    </joint>
+  </xacro:macro>
+  <xacro:macro name="knee_to_shin" params="side">
+    <joint name="knee_to_shin_${side}" type="continuous">
       <origin xyz="0.0607 0.0474 0" rpy="0 0 0"/>
       <axis xyz="0 0 1"/>
       <parent link="${side}_knee" />
       <child link="${side}_shin" />
-	  <limit lower="0" upper="0" effort="0" velocity="0" />
+      <limit lower="-100" upper="100" effort="0" velocity="100" />
     </joint>
   </xacro:macro>
@@ -321,5 +321,5 @@
       <parent link="${side}_shin" />
       <child link="${side}_tarsus" />
-	  <limit lower="-100" upper="100" effort="0" velocity="100" />
+      <limit lower="-100" upper="100" effort="0" velocity="100" />
     </joint>
   </xacro:macro>
@@ -330,5 +330,5 @@
       <parent link="${side}_tarsus" />
       <child link="${side}_toe" />
-	  <limit lower="-2.4435" upper="-0.5236" effort="0.9" velocity="11.5192" />
+      <limit lower="-2.4435" upper="-0.5236" effort="0.9" velocity="11.5192" />
     </joint>
   </xacro:macro>
