Commit message: updated urdf file to include transmissions and limits

File: urdf/cassie.urdf (robot description, URDF)
Before this commit: robot cassie_simple, 17 links, 16 joints
Joints:
- joint ankle_joint_left: limit (none) -> lower=-100 upper=100 effort=0 velocity=100
- joint ankle_joint_right: limit (none) -> lower=-100 upper=100 effort=0 velocity=100
- joint fixed_knee_to_shin_left: limit (none) -> lower=0 upper=0 effort=0 velocity=0
- joint fixed_knee_to_shin_right: limit (none) -> lower=0 upper=0 effort=0 velocity=0
- joint fixed_left: limit (none) -> lower=0 upper=0 effort=0 velocity=0
- joint fixed_right: limit (none) -> lower=0 upper=0 effort=0 velocity=0
- joint hip_abduction_left: limit (none) -> lower=-0.2618 upper=0.3927 effort=4.5 velocity=12.1475
- joint hip_abduction_right: limit (none) -> lower=-0.3927 upper=0.2618 effort=4.5 velocity=12.1475
- joint hip_flexion_left: limit (none) -> lower=-0.8727 upper=1.3963 effort=12.2 velocity=8.5085
- joint hip_flexion_right: limit (none) -> lower=-0.8727 upper=1.3963 effort=12.2 velocity=8.5085
- joint hip_rotation_left: limit (none) -> lower=-0.3927 upper=0.3927 effort=4.5 velocity=12.1475
- joint hip_rotation_right: limit (none) -> lower=-0.3927 upper=0.3927 effort=4.5 velocity=12.1475
- joint knee_joint_left: limit (none) -> lower=-2.8623 upper=-0.6458 effort=12.2 velocity=8.5085
- joint knee_joint_right: limit (none) -> lower=-2.8623 upper=-0.6458 effort=12.2 velocity=8.5085
- joint toe_joint_left: limit (none) -> lower=-2.4435 upper=-0.5236 effort=0.9 velocity=11.5192
- joint toe_joint_right: limit (none) -> lower=-2.4435 upper=-0.5236 effort=0.9 velocity=11.5192

File: urdf/cassie.xacro (robot description, xacro)
@@ -47,4 +47,15 @@
   <xacro:ankle_joint side="right"/>
   <xacro:toe_joint side="right"/>
+  <!-- Transmissions -->
+  <xacro:hip_abduction_trans side="left"/>
+  <xacro:hip_rotation_trans side="left"/>
+  <xacro:hip_flexion_trans side="left"/>
+  <xacro:knee_joint_trans side="left"/>
+  <xacro:toe_joint_trans side="left"/>
+  <xacro:hip_abduction_trans side="right"/>
+  <xacro:hip_rotation_trans side="right"/>
+  <xacro:hip_flexion_trans side="right"/>
+  <xacro:knee_joint_trans side="right"/>
+  <xacro:toe_joint_trans side="right"/>
   <!-- Link Definitions-->
   <xacro:macro name="pelvis" params="cname color">
@@ -217,4 +228,5 @@
       <parent link="pelvis" />
       <child link="${side}_pelvis_abduction" />
+	  <limit lower="0" upper="0" effort="0" velocity="0" />
     </joint>
   </xacro:macro>
@@ -225,4 +237,10 @@
       <parent link="${side}_pelvis_abduction" />
       <child link="${side}_pelvis_rotation" />
+	  <xacro:if value="${side == 'left'}">
+	    <limit lower="-0.2618" upper="0.3927" effort="4.5" velocity="12.1475" />
+	  </xacro:if>
+	  <xacro:if value="${side == 'right'}">
+	    <limit lower="-0.3927" upper="0.2618" effort="4.5" velocity="12.1475" />
+	  </xacro:if>
     </joint>
   </xacro:macro>
@@ -233,4 +251,5 @@
       <parent link="${side}_pelvis_rotation" />
       <child link="${side}_hip" />
+	  <limit lower="-0.3927" upper="0.3927" effort="4.5" velocity="12.1475" />
     </joint>
   </xacro:macro>
@@ -241,4 +260,5 @@
       <parent link="${side}_hip" />
       <child link="${side}_thigh" />
+	  <limit lower="-0.8727" upper="1.3963" effort="12.2" velocity="8.5085" />
     </joint>
   </xacro:macro>
@@ -249,4 +269,5 @@
       <parent link="${side}_thigh" />
       <child link="${side}_knee" />
+	  <limit lower="-2.8623" upper="-0.6458" effort="12.2" velocity="8.5085" />
     </joint>
   </xacro:macro>
@@ -257,4 +278,5 @@
       <parent link="${side}_knee" />
       <child link="${side}_shin" />
+	  <limit lower="0" upper="0" effort="0" velocity="0" />
     </joint>
   </xacro:macro>
@@ -265,4 +287,5 @@
       <parent link="${side}_shin" />
       <child link="${side}_tarsus" />
+	  <limit lower="-100" upper="100" effort="0" velocity="100" />
     </joint>
   </xacro:macro>
@@ -273,5 +296,47 @@
       <parent link="${side}_tarsus" />
       <child link="${side}_toe" />
-    </joint>
+	  <limit lower="-2.4435" upper="-0.5236" effort="0.9" velocity="11.5192" />
+    </joint>
+  </xacro:macro>
+  <!-- Transmission Definitions -->
+  <xacro:macro name="hip_abduction_trans" params="side">
+    <transmission name="hip_abduction_trans_${side}" type="transmission_interface/SimpleTransmission">
+	  <joint name="hip_abduction_${side}"/>
+	  <actuator name="hip_abduction_motor_${side}"/>
+	  <actuatorInertia>0.000061</actuatorInertia>
+	  <mechanicalReduction>25</mechanicalReduction>
+    </transmission>
+  </xacro:macro>
+  <xacro:macro name="hip_rotation_trans" params="side">
+    <transmission name="hip_rotation_trans_${side}" type="transmission_interface/SimpleTransmission">
+	  <joint name="hip_rotation_${side}"/>
+	  <actuator name="hip_rotation_motor_${side}"/>
+	  <actuatorInertia>0.000061</actuatorInertia>
+	  <mechanicalReduction>25</mechanicalReduction>
+    </transmission>
+  </xacro:macro>
+  <xacro:macro name="hip_flexion_trans" params="side">
+    <transmission name="hip_flexion_trans_${side}" type="transmission_interface/SimpleTransmission">
+	  <joint name="hip_flexion_${side}"/>
+	  <actuator name="hip_flexion_motor_${side}"/>
+	  <actuatorInertia>0.000365</actuatorInertia>
+	  <mechanicalReduction>16</mechanicalReduction>
+    </transmission>
+  </xacro:macro>
+  <xacro:macro name="knee_joint_trans" params="side">
+    <transmission name="knee_joint_trans_${side}" type="transmission_interface/SimpleTransmission">
+	  <joint name="knee_joint_${side}"/>
+	  <actuator name="knee_joint_motor_${side}"/>
+	  <actuatorInertia>0.000365</actuatorInertia>
+	  <mechanicalReduction>16</mechanicalReduction>
+    </transmission>
+  </xacro:macro>
+  <xacro:macro name="toe_joint_trans" params="side">
+    <transmission name="toe_joint_trans_${side}" type="transmission_interface/SimpleTransmission">
+	  <joint name="toe_joint_${side}"/>
+	  <actuator name="toe_joint_motor_${side}"/>
+	  <actuatorInertia>0.0000049</actuatorInertia>
+	  <mechanicalReduction>50</mechanicalReduction>
+    </transmission>
   </xacro:macro>
 </robot>

Commit message: Modified launch file so joint state gui is opened by default

File: urdf/cassie.urdf (robot description, URDF)
Before this commit: robot cassie_simple, 17 links, 16 joints
Joints:
- joint hip_rotation_left: axis 1 0 0 -> -1 0 0
- joint hip_rotation_right: axis 1 0 0 -> -1 0 0

File: urdf/cassie.xacro (robot description, xacro)
@@ -3,5 +3,5 @@
 	 Email:  rosshart@umich.edu
      Date:   04/24/2016   -->
-<robot name="cassie_simple"
+<robot name="cassie"
   xmlns:xacro="http://ros.org/wiki/xacro">
   <!-- Properties -->
@@ -248,5 +248,5 @@
     <joint name="hip_rotation_${side}" type="continuous">
       <origin xyz="0 0 -0.09" rpy="0 ${pi/2} ${-pi/2}"/>
-      <axis xyz="1 0 0"/>
+      <axis xyz="-1 0 0"/>
       <parent link="${side}_pelvis_rotation" />
       <child link="${side}_hip" />
@@ -304,5 +304,5 @@
 	  <joint name="hip_abduction_${side}"/>
 	  <actuator name="hip_abduction_motor_${side}"/>
-	  <actuatorInertia>0.000061</actuatorInertia>
+	  <motorInertia>0.000061</motorInertia>
 	  <mechanicalReduction>25</mechanicalReduction>
     </transmission>
@@ -312,5 +312,5 @@
 	  <joint name="hip_rotation_${side}"/>
 	  <actuator name="hip_rotation_motor_${side}"/>
-	  <actuatorInertia>0.000061</actuatorInertia>
+	  <motorInertia>0.000061</motorInertia>
 	  <mechanicalReduction>25</mechanicalReduction>
     </transmission>
@@ -320,5 +320,5 @@
 	  <joint name="hip_flexion_${side}"/>
 	  <actuator name="hip_flexion_motor_${side}"/>
-	  <actuatorInertia>0.000365</actuatorInertia>
+	  <motorInertia>0.000365</motorInertia>
 	  <mechanicalReduction>16</mechanicalReduction>
     </transmission>
@@ -328,5 +328,5 @@
 	  <joint name="knee_joint_${side}"/>
 	  <actuator name="knee_joint_motor_${side}"/>
-	  <actuatorInertia>0.000365</actuatorInertia>
+	  <motorInertia>0.000365</motorInertia>
 	  <mechanicalReduction>16</mechanicalReduction>
     </transmission>
@@ -336,5 +336,5 @@
 	  <joint name="toe_joint_${side}"/>
 	  <actuator name="toe_joint_motor_${side}"/>
-	  <actuatorInertia>0.0000049</actuatorInertia>
+	  <motorInertia>0.0000049</motorInertia>
 	  <mechanicalReduction>50</mechanicalReduction>
     </transmission>

Commit message: updated urdfs and launch file

File: urdf/cassie.urdf (robot description, URDF)
Before this commit: robot cassie, 17 links, 16 joints
Links:
- added link vectorNav, mass 0
Joints:
- removed joint fixed_knee_to_shin_left
- removed joint fixed_knee_to_shin_right
- added joint fixed_pelvis_to_vectorNav: type fixed, parent pelvis, child vectorNav, origin xyz=0.03155 0 -0.07996 rpy=0 0 0
- added joint knee_to_shin_left: type continuous, parent left_knee, child left_shin, origin xyz=0.0607 0.0474 0 rpy=0 0 0, axis 0 0 1, limit lower=-100 upper=100 effort=0 velocity=100
- added joint knee_to_shin_right: type continuous, parent right_knee, child right_shin, origin xyz=0.0607 0.0474 0 rpy=0 0 0, axis 0 0 1, limit lower=-100 upper=100 effort=0 velocity=100
- joint fixed_left: axis 0 0 1 -> (none); limit lower=0 upper=0 effort=0 velocity=0 -> (none)
- joint fixed_right: axis 0 0 1 -> (none); limit lower=0 upper=0 effort=0 velocity=0 -> (none)

File: urdf/cassie.xacro (robot description, xacro)
@@ -13,4 +13,5 @@
   <xacro:property name="light_grey_RGB" value="0.75 0.75 0.75 1" />
   <!-- Links -->
+  <xacro:vectorNav />
   <xacro:pelvis cname="grey" color="${grey_RGB}" />
   <xacro:pelvis_abduction side="left" cname="light_grey" color="${light_grey_RGB}" stl_ext=""/>
@@ -31,4 +32,5 @@
   <xacro:toe side="right" cname="light_grey" color="${light_grey_RGB}" stl_ext="_mirror" reflect="-1"/>
   <!-- Joints -->
+  <xacro:fixed_pelvis_to_vectorNav />
   <xacro:fixed_pelvis_to_abduction side="left" reflect="1"/>
   <xacro:hip_abduction side="left"/>
@@ -36,5 +38,5 @@
   <xacro:hip_flexion side="left"/>
   <xacro:knee_joint side="left" reflect="1"/>
-  <xacro:fixed_knee_to_shin side="left"/>
+  <xacro:knee_to_shin side="left"/>
   <xacro:ankle_joint side="left"/>
   <xacro:toe_joint side="left"/>
@@ -44,5 +46,5 @@
   <xacro:hip_flexion side="right"/>
   <xacro:knee_joint side="right" reflect="-1"/>
-  <xacro:fixed_knee_to_shin side="right"/>
+  <xacro:knee_to_shin side="right"/>
   <xacro:ankle_joint side="right"/>
   <xacro:toe_joint side="right"/>
@@ -59,4 +61,13 @@
   <xacro:toe_joint_trans side="right"/>
   <!-- Link Definitions-->
+  <xacro:macro name="vectorNav">
+    <link name="vectorNav">
+      <inertial>
+        <origin xyz="0 0 0" rpy="0 0 0"/>
+        <mass value="0" />
+                <inertia ixx="0" ixy="0" ixz="0" iyy="0" iyz="0" izz="0" />
+      </inertial>
+    </link>
+  </xacro:macro>
   <xacro:macro name="pelvis" params="cname color">
     <link name="pelvis">
@@ -222,11 +233,16 @@
   </xacro:macro>
   <!-- Joint Definitions -->
+  <xacro:macro name="fixed_pelvis_to_vectorNav">
+    <joint name="fixed_pelvis_to_vectorNav" type="fixed">
+      <origin xyz="0.03155 0 -0.07996" rpy="0 0 0"/>
+      <parent link="pelvis" />
+      <child link="vectorNav" />
+    </joint>
+  </xacro:macro>
   <xacro:macro name="fixed_pelvis_to_abduction" params="side reflect">
     <joint name="fixed_${side}" type="fixed">
       <origin xyz="0.021 ${reflect*0.135} 0" rpy="0 ${pi/2} 0"/>
-      <axis xyz="0 0 1"/>
       <parent link="pelvis" />
       <child link="${side}_pelvis_abduction" />
-	  <limit lower="0" upper="0" effort="0" velocity="0" />
     </joint>
   </xacro:macro>
@@ -251,5 +267,5 @@
       <parent link="${side}_pelvis_rotation" />
       <child link="${side}_hip" />
-	  <limit lower="-0.3927" upper="0.3927" effort="4.5" velocity="12.1475" />
+      <limit lower="-0.3927" upper="0.3927" effort="4.5" velocity="12.1475" />
     </joint>
   </xacro:macro>
@@ -260,5 +276,5 @@
       <parent link="${side}_hip" />
       <child link="${side}_thigh" />
-	  <limit lower="-0.8727" upper="1.3963" effort="12.2" velocity="8.5085" />
+      <limit lower="-0.8727" upper="1.3963" effort="12.2" velocity="8.5085" />
     </joint>
   </xacro:macro>
@@ -269,14 +285,14 @@
       <parent link="${side}_thigh" />
       <child link="${side}_knee" />
-	  <limit lower="-2.8623" upper="-0.6458" effort="12.2" velocity="8.5085" />
-    </joint>
-  </xacro:macro>
-  <xacro:macro name="fixed_knee_to_shin" params="side">
-    <joint name="fixed_knee_to_shin_${side}" type="fixed">
+      <limit lower="-2.8623" upper="-0.6458" effort="12.2" velocity="8.5085" />
+    </joint>
+  </xacro:macro>
+  <xacro:macro name="knee_to_shin" params="side">
+    <joint name="knee_to_shin_${side}" type="continuous">
       <origin xyz="0.0607 0.0474 0" rpy="0 0 0"/>
       <axis xyz="0 0 1"/>
       <parent link="${side}_knee" />
       <child link="${side}_shin" />
-	  <limit lower="0" upper="0" effort="0" velocity="0" />
+      <limit lower="-100" upper="100" effort="0" velocity="100" />
     </joint>
   </xacro:macro>
@@ -287,5 +303,5 @@
       <parent link="${side}_shin" />
       <child link="${side}_tarsus" />
-	  <limit lower="-100" upper="100" effort="0" velocity="100" />
+      <limit lower="-100" upper="100" effort="0" velocity="100" />
     </joint>
   </xacro:macro>
@@ -296,5 +312,5 @@
       <parent link="${side}_tarsus" />
       <child link="${side}_toe" />
-	  <limit lower="-2.4435" upper="-0.5236" effort="0.9" velocity="11.5192" />
+      <limit lower="-2.4435" upper="-0.5236" effort="0.9" velocity="11.5192" />
     </joint>
   </xacro:macro>

File: urdf/cassie_with_base.urdf (robot description, URDF)
Before this commit: robot cassie, 25 links, 24 joints
Links:
- removed link multisense
Joints:
- removed joint fixed_pelvis_to_multisense
- joint fixed_pelvis_to_vectorNav: origin xyz=0.03155 0 -0.07996 rpy=3.14159265359 0 0 -> xyz=0.03155 0 -0.07996 rpy=0 0 0

File: urdf/cassie_with_base.xacro (robot description, xacro)
@@ -19,5 +19,4 @@
   <xacro:yaw_link />
   <xacro:pitch_link />
-  <xacro:multisense />
   <xacro:vectorNav />
   <xacro:pelvis cname="grey" color="${grey_RGB}" />
@@ -45,5 +44,4 @@
   <xacro:pitch />
   <xacro:roll />
-  <xacro:fixed_pelvis_to_multisense />
   <xacro:fixed_pelvis_to_vectorNav />
   <xacro:fixed_pelvis_to_abduction side="left" reflect="1"/>
@@ -129,13 +127,4 @@
     </link>
   </xacro:macro>
-  <xacro:macro name="multisense">
-    <link name="multisense">
-      <inertial>
-        <origin xyz="0 0 0.25" rpy="0 0 0"/>
-        <mass value="0" />
-                <inertia ixx="0" ixy="0" ixz="0" iyy="0" iyz="0" izz="0" />
-      </inertial>
-    </link>
-  </xacro:macro>
   <xacro:macro name="vectorNav">
     <link name="vectorNav">
@@ -361,14 +350,7 @@
     </joint>
   </xacro:macro>
-  <xacro:macro name="fixed_pelvis_to_multisense">
-    <joint name="fixed_pelvis_to_multisense" type="fixed">
-      <origin xyz="0 0 0.25" rpy="0 0 0"/>
-      <parent link="pelvis" />
-      <child link="multisense" />
-    </joint>
-  </xacro:macro>
   <xacro:macro name="fixed_pelvis_to_vectorNav">
     <joint name="fixed_pelvis_to_vectorNav" type="fixed">
-      <origin xyz="0.03155 0 -0.07996" rpy="${pi} 0 0"/>
+      <origin xyz="0.03155 0 -0.07996" rpy="0 0 0"/>
       <parent link="pelvis" />
       <child link="vectorNav" />
