Commit message: changed torso mesh name

File: urdf/cassie_with_torso.urdf (robot description, URDF)
Before this commit: robot cassie, 23 links, 22 joints
Links:
- link torso: geometry visual mesh filename=package://cassie_description/meshes/torso.stl scale=0.001 0.001 0.001

Commit message: added reduced torso mesh

File: urdf/cassie_with_torso.urdf (robot description, URDF)
Before this commit: robot cassie, 23 links, 22 joints
Joints:
- removed joint fixed_torso_to_pelvis
- added joint fixed_pelvis_to_torso: type fixed, parent pelvis, child torso, origin xyz=0 0 0.15 rpy=0 0 0

File: urdf/cassie_with_torso.xacro (robot description, xacro)
@@ -276,9 +276,9 @@
   </xacro:macro>
   <!-- Joint Definitions -->
-  <xacro:macro name="fixed_torso_to_pelvis">
-    <joint name="fixed_torso_to_pelvis" type="fixed">
-      <origin xyz="0 0 -0.15" rpy="0 0 0"/>
-      <parent link="torso" />
-      <child link="pelvis" />
+  <xacro:macro name="fixed_pelvis_to_torso">
+    <joint name="fixed_pelvis_to_torso" type="fixed">
+      <origin xyz="0 0 0.15" rpy="0 0 0"/>
+      <parent link="pelvis" />
+      <child link="torso" />
     </joint>
   </xacro:macro>
@@ -459,5 +459,5 @@
   <xacro:toe side="right" cname="light_grey" color="${light_grey_RGB}" stl_ext="_mirror" reflect="-1"/>
   <!-- Joints -->
-  <xacro:fixed_torso_to_pelvis/>
+  <xacro:fixed_pelvis_to_torso/>
   <xacro:fixed_torso_to_top_lidar/>
   <xacro:fixed_torso_to_tilted_lidar/>

Commit message: Changed torso origin to a better location. Visualization does not need extra transformation and rotations now

File: urdf/cassie_with_torso.urdf (robot description, URDF)
Before this commit: robot cassie, 23 links, 22 joints
Links:
- link torso: geometry visual mesh filename=package://cassie_description/meshes/torso.stl scale=1 1 1
Joints:
- joint fixed_pelvis_to_torso: origin xyz=0 0 0.15 rpy=0 0 0 -> xyz=0.0218 0 0.2606 rpy=0 0 0
- joint fixed_torso_to_back_camera: origin xyz=-0.12 0 0.19 rpy=0 0 3.14 -> xyz=-0.1418 0 0.07 rpy=0 0 3.14
- joint fixed_torso_to_front_camera: origin xyz=0.16 0 0.19 rpy=0 0 0 -> xyz=0.1382 0 0.07 rpy=0 0 0
- joint fixed_torso_to_tilted_lidar: origin xyz=0.14 0 0.25 rpy=0 0.65 0 -> xyz=0.1182 0 0.13 rpy=0 0.65 0
- joint fixed_torso_to_top_lidar: origin xyz=0.065 0 0.38 rpy=0 0 0 -> xyz=0.0432 0 0.27 rpy=0 0 0

File: urdf/cassie_with_torso.xacro (robot description, xacro)
@@ -22,7 +22,7 @@
       </inertial>
       <visual>
-          <origin xyz="-0.192 -0.19 -0.095" rpy="1.57 0 1.57" />
-        <geometry>
-          <mesh filename="package://cassie_description/meshes/CassieTorso_Mount.STL" scale="0.001 0.001 0.001"/>
+          <origin xyz="0 0 0" rpy="0 0 0" />
+        <geometry>
+          <mesh filename="package://cassie_description/meshes/torso.stl" scale="1 1 1"/>
         </geometry>
         <material name="${cname}">
@@ -278,5 +278,5 @@
   <xacro:macro name="fixed_pelvis_to_torso">
     <joint name="fixed_pelvis_to_torso" type="fixed">
-      <origin xyz="0 0 0.15" rpy="0 0 0"/>
+      <origin xyz="0.0218 0 0.2606" rpy="0 0 0"/>
       <parent link="pelvis" />
       <child link="torso" />
@@ -285,5 +285,5 @@
   <xacro:macro name="fixed_torso_to_top_lidar">
     <joint name="fixed_torso_to_top_lidar" type="fixed">
-      <origin xyz="0.065 0 0.38" rpy="0 0 0"/>
+      <origin xyz="0.0432 0 0.27" rpy="0 0 0"/>
       <parent link="torso" />
       <child link="top_lidar" />
@@ -292,5 +292,5 @@
   <xacro:macro name="fixed_torso_to_tilted_lidar">
     <joint name="fixed_torso_to_tilted_lidar" type="fixed">
-      <origin xyz="0.14 0 0.25" rpy="0 0.65 0"/>
+      <origin xyz="0.1182 0 0.13" rpy="0 0.65 0"/>
       <parent link="torso" />
       <child link="tilted_lidar" />
@@ -299,5 +299,5 @@
   <xacro:macro name="fixed_torso_to_front_camera">
     <joint name="fixed_torso_to_front_camera" type="fixed">
-      <origin xyz="0.16 0 0.19" rpy="0 0 0"/>
+      <origin xyz="0.1382 0 0.07" rpy="0 0 0"/>
       <parent link="torso" />
       <child link="front_camera" />
@@ -306,5 +306,5 @@
   <xacro:macro name="fixed_torso_to_back_camera">
     <joint name="fixed_torso_to_back_camera" type="fixed">
-      <origin xyz="-0.12 0 0.19" rpy="0 0 3.14"/>
+      <origin xyz="-0.1418 0 0.07" rpy="0 0 3.14"/>
       <parent link="torso" />
       <child link="back_camera" />

File: urdf/torso.urdf (robot description, URDF)
Before this commit: robot cassie, 5 links, 4 joints
Links:
- link torso: geometry visual mesh filename=package://cassie_description/meshes/torso.stl scale=1 1 1
Joints:
- joint fixed_torso_to_back_camera: origin xyz=-0.12 0 0.19 rpy=0 0 3.14 -> xyz=-0.1418 0 0.07 rpy=0 0 3.14
- joint fixed_torso_to_front_camera: origin xyz=0.16 0 0.19 rpy=0 0 0 -> xyz=0.1382 0 0.07 rpy=0 0 0
- joint fixed_torso_to_tilted_lidar: origin xyz=0.14 0 0.25 rpy=0 0.65 0 -> xyz=0.1182 0 0.13 rpy=0 0.65 0
- joint fixed_torso_to_top_lidar: origin xyz=0.065 0 0.38 rpy=0 0 0 -> xyz=0.0432 0 0.27 rpy=0 0 0

Commit message: updated inertia properties for torso

File: urdf/cassie_with_torso.urdf (robot description, URDF)
Before this commit: robot cassie, 23 links, 22 joints
Links:
- link torso: mass 8 -> 8.5

File: urdf/cassie_with_torso.xacro (robot description, xacro)
@@ -17,6 +17,6 @@
     <link name="torso">
       <inertial>
-        <origin xyz="0 0 0" rpy="0 0 0"/>
-        <mass value="8" />
+      <origin rpy="0 0 0" xyz="0.00637 -0.00235 0.0803"/>
+      <mass value="8.5"/>
 		<inertia ixx=".0942" ixy=".000169" ixz=".015" iyy=".084" iyz=".000516" izz=".113" />
       </inertial>

File: urdf/torso.urdf (robot description, URDF)
Before this commit: robot cassie, 5 links, 4 joints
Links:
- link torso: mass 8 -> 8.5
